File: prototype/kicad/a3982slb_board.sch (KiCad schematic (older format))
At the start: 16 parts, among them P1 CONN_01X07, P2 CONN_01X06, U1 A3982

Commit message: Routing completed.
Parts:
- C4: footprint (none) -> wshito_FootPrints:UCB1H101MNL1GS_HandSoldering
- R1, R2: footprint (none) -> Resistors_SMD:R_2512_HandSoldering
- R3: footprint (none) -> Resistors_SMD:R_0603_HandSoldering; Power 1/8W -> 1/10W
- R4: footprint (none) -> Resistors_SMD:R_0603_HandSoldering
- RV1: footprint (none) -> wshito_FootPrints:G43A
- U1: footprint (none) -> Housings_SOIC:SOIC-24W_7.5x15.4mm_Pitch1.27mm
- W1: footprint (none) -> Measurement_Points:Measurement_Point_Square-TH_Small
Connections:
- net +3V3: now also RV1.1; no longer RV1.3
- net DIR: now also P1.5 (P5); no longer P1.4 (P4)
- net ENABLE: now also P2.5 (P5); no longer P1.7 (P7)
- net GND: now also P1.4 (P4), P2.4 (P4); no longer P1.2 (P2), P2.2 (P2)
- net MS1: now also P2.6 (P6); no longer P1.6 (P6)
- net OUT1A: now also P1.7 (P7); no longer P2.3 (P3)
- net OUT1B: now also P1.6 (P6); no longer P2.4 (P4)
- net OUT2A: now also P2.2 (P2); no longer P2.5 (P5)
- net OUT2B: now also P2.3 (P3); no longer P2.6 (P6)
- net RESET: now also P1.2 (P2); no longer P1.5 (P5)
- net at R4.1: now also RV1.3; no longer RV1.1
Other:
- note added: "Swapped the pin in schematic. \nThe top pin is the pin 1."
Changed lines of the file:
@@
 EESchema Schematic File Version 2
-LIBS:a3982slb_board-rescue
+LIBS:wshito
 LIBS:power
 LIBS:device
@@
 LIBS:valves
 LIBS:motor_driver
-LIBS:wshito
 LIBS:a3982slb_board-cache
 EELAYER 25 0
@@
 Comment4 ""
 $EndDescr
-Text GLabel 9500 1900 0    60   Input ~ 0
+Text GLabel 9500 1600 0    60   Input ~ 0
 OUT2A
 Text GLabel 5550 3950 0    60   Output ~ 0
@@
 Text GLabel 7250 4250 2    60   Output ~ 0
 OUT1B
-Text GLabel 9500 2000 0    60   Input ~ 0
+Text GLabel 9500 1700 0    60   Input ~ 0
 OUT2B
-Text GLabel 9500 1700 0    60   Input ~ 0
+Text GLabel 7450 2100 0    60   Input ~ 0
 OUT1A
-Text GLabel 9500 1800 0    60   Input ~ 0
+Text GLabel 7450 2000 0    60   Input ~ 0
 OUT1B
 Text GLabel 7250 4850 2    60   Input ~ 0
@@
 F 0 "W1" H 8900 4820 50  0000 C CNN
 F 1 "TEST_1P" H 8900 4750 50  0000 C CNN
-F 2 "" H 9100 4550 50  0001 C CNN
+F 2 "Measurement_Points:Measurement_Point_Square-TH_Small" H 9100 4550 50  0001 C CNN
 F 3 "" H 9100 4550 50  0000 C CNN
 	1    8900 4550
@@
 F 0 "RV1" V 9125 4650 50  0000 C CNN
 F 1 "10K" V 9200 4650 50  0000 C CNN
-F 2 "" H 9300 4650 50  0001 C CNN
+F 2 "wshito_FootPrints:G43A" H 9300 4650 50  0001 C CNN
 F 3 "" H 9300 4650 50  0000 C CNN
 	1    9300 4650
-	-1   0    0    1
+	-1   0    0    -1
 $EndComp
 Text GLabel 9300 4250 1    60   Input ~ 0
@@
 F 0 "R1" V 4380 4050 50  0000 C CNN
 F 1 "0.33" V 4300 4050 50  0000 C CNN
-F 2 "" V 4230 4050 50  0001 C CNN
+F 2 "Resistors_SMD:R_2512_HandSoldering" V 4230 4050 50  0001 C CNN
 F 3 "" V 4380 4050 50  0000 C CNN
 F 4 "2W" V 4220 4050 50  0000 C CNN "Power"
@@
 F 0 "R2" V 8030 4150 50  0000 C CNN
 F 1 "0.33" V 7950 4150 50  0000 C CNN
-F 2 "" V 7880 4150 50  0001 C CNN
+F 2 "Resistors_SMD:R_2512_HandSoldering" V 7880 4150 50  0001 C CNN
 F 3 "" V 8030 4150 50  0000 C CNN
 F 4 "2W" V 7870 4150 50  0000 C CNN "Power"
@@
 F 0 "R4" V 9380 5400 50  0000 C CNN
 F 1 "2.4K" V 9300 5400 50  0000 C CNN
-F 2 "" V 9230 5400 50  0001 C CNN
+F 2 "Resistors_SMD:R_0603_HandSoldering" V 9230 5400 50  0001 C CNN
 F 3 "" V 9380 5400 50  0000 C CNN
 F 4 "1/8W" V 9220 5400 50  0000 C CNN "Power"
@@
 F 0 "R3" V 8030 4750 50  0000 C CNN
 F 1 "25K" V 7950 4750 50  0000 C CNN
-F 2 "" V 7880 4750 50  0001 C CNN
+F 2 "Resistors_SMD:R_0603_HandSoldering" V 7880 4750 50  0001 C CNN
 F 3 "" V 8030 4750 50  0000 C CNN
-F 4 "1/8W" V 7870 4750 50  0000 C CNN "Power"
+F 4 "1/10W" V 7870 4750 50  0000 C CNN "Power"
 	1    7950 4750
 	-1   0    0    1
@@
 F 0 "C4" H 6910 3170 50  0000 L CNN
 F 1 "100u" H 6910 3020 50  0000 L CNN
-F 2 "" H 6900 3100 50  0001 C CNN
+F 2 "wshito_FootPrints:UCB1H101MNL1GS_HandSoldering" H 6900 3100 50  0001 C CNN
 F 3 "" H 6900 3100 50  0000 C CNN
 F 4 "50V" H 6890 3020 50  0000 R CNN "Voltage"
@@
 	1    0    0    -1
 $EndComp
-Wire Wire Line
-	5750 3950 5550 3950
-Wire Wire Line
-	7050 3950 7250 3950
-Wire Wire Line
-	7050 4250 7250 4250
-Wire Wire Line
-	5750 4250 5550 4250
-Wire Wire Line
-	7050 4850 7250 4850
-Wire Wire Line
-	7050 4650 9150 4650
-Wire Wire Line
-	9300 4800 9300 5250
-Wire Wire Line
-	9300 5550 9300 5800
-Wire Wire Line
-	9300 4500 9300 4250
-Connection ~ 8900 4650
-Wire Wire Line
-	8900 4650 8900 4550
-Wire Wire Line
-	5750 4050 4450 4050
-Wire Wire Line
-	4150 4050 3200 4050
-Wire Wire Line
-	7050 4150 7800 4150
-Wire Wire Line
-	8100 4150 8550 4150
-Wire Wire Line
-	8550 4150 8550 5800
-Wire Wire Line
-	3200 4050 3200 5800
-Wire Wire Line
-	3200 4450 5750 4450
-Connection ~ 3200 4450
-Wire Wire Line
-	5750 4650 5600 4650
-Wire Wire Line
-	5400 4650 5250 4650
-Wire Wire Line
-	5250 4650 5250 4750
-Wire Wire Line
-	5250 4750 5750 4750
-Wire Wire Line
-	7050 4350 7250 4350
-Wire Wire Line
-	7050 4750 7250 4750
-Wire Wire Line
-	5750 4350 5550 4350
-Wire Wire Line
-	5750 5050 5550 5050
-Wire Wire Line
-	7050 4950 7950 4950
-Wire Wire Line
-	7050 4550 8200 4550
-Wire Wire Line
-	7050 4450 8550 4450
-Connection ~ 8550 4450
-Wire Wire Line
-	8200 4550 8200 5800
-Connection ~ 7950 4550
-Wire Wire Line
-	7050 5050 7250 5050
-Wire Wire Line
-	7150 4850 7150 5600
-Wire Wire Line
-	7150 5600 7500 5600
-Connection ~ 7150 4850
-Wire Wire Line
-	7700 5600 8200 5600
-Connection ~ 8200 5600
-Wire Wire Line
-	7150 5300 7500 5300
-Connection ~ 7150 5300
-Wire Wire Line
-	7700 5300 8200 5300
-Connection ~ 8200 5300
-Wire Wire Line
-	5750 4150 4800 4150
-Wire Wire Line
-	4800 3550 4800 4600
-Wire Wire Line
-	4800 4800 4800 4850
-Wire Wire Line
-	4800 4850 5750 4850
-Wire Wire Line
-	6400 2900 6400 3650
-Wire Wire Line
-	6400 3100 6800 3100
-Connection ~ 6400 3100
-Wire Wire Line
-	6800 3350 6400 3350
-Connection ~ 6400 3350
-Wire Wire Line
-	7000 3350 7900 3350
-Wire Wire Line
-	7900 3100 7900 3750
-Wire Wire Line
-	7000 3100 7900 3100
-Connection ~ 7900 3350
-Wire Wire Line
-	7950 4550 7950 4600
-Wire Wire Line
-	7950 4950 7950 4900
-Wire Wire Line
-	5750 4550 3900 4550
-Wire Wire Line
-	3900 4550 3900 5800
-Wire Wire Line
-	5750 4950 5200 4950
-Wire Wire Line
-	5000 4950 3900 4950
-Connection ~ 3900 4950
-Wire Wire Line
-	9850 1700 9500 1700
-Wire Wire Line
-	9850 1800 9500 1800
-Wire Wire Line
-	9850 1900 9500 1900
-Wire Wire Line
-	9850 2000 9500 2000
-Wire Wire Line
-	7750 1700 7450 1700
-Wire Wire Line
-	7750 1800 7450 1800
-Wire Wire Line
-	7750 1900 7450 1900
-Wire Wire Line
-	7750 2000 7450 2000
-Wire Wire Line
-	7750 2100 7450 2100
 Text GLabel 7450 1700 0    60   Input ~ 0
 STEP
-Text GLabel 7450 1800 0    60   Input ~ 0
+Text GLabel 7450 1900 0    60   Input ~ 0
 DIR
-Text GLabel 7450 1900 0    60   Input ~ 0
+Text GLabel 7450 1600 0    60   Input ~ 0
 RESET
-Text GLabel 7450 2000 0    60   Input ~ 0
+Text GLabel 9500 2000 0    60   Input ~ 0
 MS1
-Text GLabel 7450 2100 0    60   Input ~ 0
+Text GLabel 9500 1900 0    60   Input ~ 0
 ENABLE
 $Comp
@@
 L GND #PWR08
 U 1 1 5917393E
-P 8950 1950
-F 0 "#PWR08" H 8950 1700 50  0001 C CNN
-F 1 "GND" H 8950 1800 50  0000 C CNN
-F 2 "" H 8950 1950 50  0000 C CNN
-F 3 "" H 8950 1950 50  0000 C CNN
-	1    8950 1950
+P 8950 2250
+F 0 "#PWR08" H 8950 2000 50  0001 C CNN
+F 1 "GND" H 8950 2100 50  0000 C CNN
+F 2 "" H 8950 2250 50  0000 C CNN
+F 3 "" H 8950 2250 50  0000 C CNN
+	1    8950 2250
 	1    0    0    -1
 $EndComp
@@
 	1    0    0    -1
 $EndComp
-Wire Wire Line
-	3050 1350 3050 1550
 Text GLabel 3050 1550 3    60   Input ~ 0
 VDD_LOGIC
@@
 F 0 "U1" H 6800 3750 60  0000 C CNN
 F 1 "A3982" H 6400 4350 60  0000 C CNN
-F 2 "" H 6500 4550 60  0001 C CNN
+F 2 "Housings_SOIC:SOIC-24W_7.5x15.4mm_Pitch1.27mm" H 6500 4550 60  0001 C CNN
 F 3 "" H 6500 4550 60  0001 C CNN
 	1    6400 4500
@@
 	1    0    0    -1
 $EndComp
-Wire Wire Line
-	3550 1350 3550 1550
 Text GLabel 3550 1550 3    60   Input ~ 0
 VBB_LOAD
@@
 	1    0    0    -1
 $EndComp
-Wire Wire Line
-	9850 1500 9500 1500
-Wire Wire Line
-	8950 1600 9850 1600
-Wire Wire Line
-	8950 1600 8950 1950
 $Comp
 L CONN_01X07 P1
@@
 $EndComp
 Wire Wire Line
+	5750 3950 5550 3950
+Wire Wire Line
+	7050 3950 7250 3950
+Wire Wire Line
+	7050 4250 7250 4250
+Wire Wire Line
+	5750 4250 5550 4250
+Wire Wire Line
+	7050 4850 7250 4850
+Wire Wire Line
+	7050 4650 9150 4650
+Wire Wire Line
+	9300 4800 9300 5250
+Wire Wire Line
+	9300 5550 9300 5800
+Wire Wire Line
+	9300 4500 9300 4250
+Connection ~ 8900 4650
+Wire Wire Line
+	8900 4650 8900 4550
+Wire Wire Line
+	5750 4050 4450 4050
+Wire Wire Line
+	4150 4050 3200 4050
+Wire Wire Line
+	7050 4150 7800 4150
+Wire Wire Line
+	8100 4150 8550 4150
+Wire Wire Line
+	8550 4150 8550 5800
+Wire Wire Line
+	3200 4050 3200 5800
+Wire Wire Line
+	3200 4450 5750 4450
+Connection ~ 3200 4450
+Wire Wire Line
+	5750 4650 5600 4650
+Wire Wire Line
+	5400 4650 5250 4650
+Wire Wire Line
+	5250 4650 5250 4750
+Wire Wire Line
+	5250 4750 5750 4750
+Wire Wire Line
+	7050 4350 7250 4350
+Wire Wire Line
+	7050 4750 7250 4750
+Wire Wire Line
+	5750 4350 5550 4350
+Wire Wire Line
+	5750 5050 5550 5050
+Wire Wire Line
+	7050 4950 7950 4950
+Wire Wire Line
+	7050 4550 8200 4550
+Wire Wire Line
+	7050 4450 8550 4450
+Connection ~ 8550 4450
+Wire Wire Line
+	8200 4550 8200 5800
+Connection ~ 7950 4550
+Wire Wire Line
+	7050 5050 7250 5050
+Wire Wire Line
+	7150 4850 7150 5600
+Wire Wire Line
+	7150 5600 7500 5600
+Connection ~ 7150 4850
+Wire Wire Line
+	7700 5600 8200 5600
+Connection ~ 8200 5600
+Wire Wire Line
+	7150 5300 7500 5300
+Connection ~ 7150 5300
+Wire Wire Line
+	7700 5300 8200 5300
+Connection ~ 8200 5300
+Wire Wire Line
+	5750 4150 4800 4150
+Wire Wire Line
+	4800 3550 4800 4600
+Wire Wire Line
+	4800 4800 4800 4850
+Wire Wire Line
+	4800 4850 5750 4850
+Wire Wire Line
+	6400 2900 6400 3650
+Wire Wire Line
+	6400 3100 6800 3100
+Connection ~ 6400 3100
+Wire Wire Line
+	6800 3350 6400 3350
+Connection ~ 6400 3350
+Wire Wire Line
+	7000 3350 7900 3350
+Wire Wire Line
+	7900 3100 7900 3750
+Wire Wire Line
+	7000 3100 7900 3100
+Connection ~ 7900 3350
+Wire Wire Line
+	7950 4550 7950 4600
+Wire Wire Line
+	7950 4950 7950 4900
+Wire Wire Line
+	5750 4550 3900 4550
+Wire Wire Line
+	3900 4550 3900 5800
+Wire Wire Line
+	5750 4950 5200 4950
+Wire Wire Line
+	5000 4950 3900 4950
+Connection ~ 3900 4950
+Wire Wire Line
+	9850 1700 9500 1700
+Wire Wire Line
+	8950 1800 9850 1800
+Wire Wire Line
+	9850 1900 9500 1900
+Wire Wire Line
+	9850 2000 9500 2000
+Wire Wire Line
+	6750 1800 7750 1800
+Wire Wire Line
+	7750 1900 7450 1900
+Wire Wire Line
+	7750 2000 7450 2000
+Wire Wire Line
+	7750 2100 7450 2100
+Wire Wire Line
+	3050 1350 3050 1550
+Wire Wire Line
+	3550 1350 3550 1550
+Wire Wire Line
+	9850 1500 9500 1500
+Wire Wire Line
 	7750 1500 7450 1500
-Wire Wire Line
-	6750 1600 7750 1600
-Wire Wire Line
-	6750 1600 6750 2050
 Wire Wire Line
 	4800 3550 6400 3550
 Connection ~ 4800 4150
 Connection ~ 6400 3550
+Text Notes 9350 4500 0    60   ~ 0
+Swapped the pin in schematic. \nThe top pin is the pin 1.
+Wire Wire Line
+	7750 1600 7450 1600
+Wire Wire Line
+	6750 1800 6750 2050
+Wire Wire Line
+	7750 1700 7450 1700
+Wire Wire Line
+	9850 1600 9500 1600
+Wire Wire Line
+	8950 1800 8950 2250
 $EndSCHEMATC
