File: prototype/kicad/a3982slb_board.kicad_pcb (KiCad board)
At the start: 2 copper layers, 21.3 x 40.9 mm, 16 parts, among them P1 CONN_01X07, P2 CONN_01X06, U1 A3982

Commit message: Silk is completed.  All done.
Parts:
- moved Test 3.24 mm to (97.2, 82.0)
- moved RV1 0.25 mm to (102.1, 82.4)
- moved C4 0.23 mm to (100.9, 53.2)
- moved R4 0.18 mm to (109.9, 83.2)
- moved C6 0.13 mm to (109.1, 77.3)
- renumbered W1 to Test
Routing:
- net Net-(RV1-Pad2): track 20.5 -> 17.5 mm
Other:
- board text added: "A3982 board"
- board text added: "DIR"
- board text added: "GND"
- board text added: "Load"
- board text added: "Logic"
- board text added: "MS1"
- board text added: "Out1A"
- board text added: "Out1B"
- board text added: "Out2B"
- board text added: "Rst"
- board text added: "Step"
- board text added: "Vbb"
- board text added: "by W.Shito"
