File: prototype/kicad/a3982slb_board/a3982slb_board.sch (KiCad schematic (older format))
At the start: 16 parts, among them P1 CONN_01X07, P2 CONN_01X06, U1 A3982

Commit message: Added BOM information on schematic.
Parts:
- C1, C3: Available at (none) -> http://akizukidenshi.com/catalog/g/gP-04940/; Model (none) -> GRM188F11H104ZA01
- C2, C5, C7: Available at (none) -> http://akizukidenshi.com/catalog/g/gP-05624/; Model (none) -> GRM188F11H224ZA01
- C4: Available at RS 280yen for 10. -> http://jp.rs-online.com/web/p/products/0269329/
- C6: Available at (none) -> http://akizukidenshi.com/catalog/g/gP-07768/; Model (none) -> GRM188R61E106MA
- R1, R2: Available at (none) -> http://jp.rs-online.com/web/p/products/7216230/; Model (none) -> Panasonic ERJ1TRQFR33U (using 1W due to the availability)
- R3: Available at (none) -> http://jp.rs-online.com/web/p/products/8626896/; Model (none) -> Panasonic ERJPA3F3002V (30KΩ)
- R4: Available at (none) -> http://jp.rs-online.com/web/p/products/8626855/; Model (none) -> Panasonic ERJPA3F2401V
- RV1: Available at (none) -> http://akizukidenshi.com/catalog/g/gP-10785/; Model (none) -> G43ATB103
- U1: Available at (none) -> http://akizukidenshi.com/catalog/g/gI-06739/; Model (none) -> A3982SLBTR-T
Changed lines of the file:
@@
 F 2 "wshito_FootPrints:G43A" H 9300 4650 50  0001 C CNN
 F 3 "" H 9300 4650 50  0000 C CNN
+F 4 "G43ATB103" V 9300 4650 60  0001 C CNN "Model"
+F 5 "http://akizukidenshi.com/catalog/g/gP-10785/" V 9300 4650 60  0001 C CNN "Available at"
 	1    9300 4650
 	-1   0    0    -1
@@
 F 3 "" V 4380 4050 50  0000 C CNN
 F 4 "2W" V 4220 4050 50  0000 C CNN "Power"
+F 5 "Panasonic ERJ1TRQFR33U (using 1W due to the availability)" V 4300 4050 60  0001 C CNN "Model"
+F 6 "http://jp.rs-online.com/web/p/products/7216230/" V 4300 4050 60  0001 C CNN "Available at"
 	1    4300 4050
 	0    1    1    0
@@
 F 3 "" V 8030 4150 50  0000 C CNN
 F 4 "2W" V 7870 4150 50  0000 C CNN "Power"
+F 5 "Panasonic ERJ1TRQFR33U (using 1W due to the availability)" V 7950 4150 60  0001 C CNN "Model"
+F 6 "http://jp.rs-online.com/web/p/products/7216230/" V 7950 4150 60  0001 C CNN "Available at"
 	1    7950 4150
 	0    1    1    0
@@
 F 3 "" V 9380 5400 50  0000 C CNN
 F 4 "1/8W" V 9220 5400 50  0000 C CNN "Power"
+F 5 "Panasonic ERJPA3F2401V" V 9300 5400 60  0001 C CNN "Model"
+F 6 "http://jp.rs-online.com/web/p/products/8626855/" V 9300 5400 60  0001 C CNN "Available at"
 	1    9300 5400
 	1    0    0    -1
@@
 F 3 "" H 5500 4650 50  0000 C CNN
 F 4 "50V" H 5480 4570 50  0000 R CNN "Voltage"
+F 5 "GRM188F11H104ZA01" H 5500 4650 60  0001 C CNN "Model"
+F 6 "http://akizukidenshi.com/catalog/g/gP-04940/" H 5500 4650 60  0001 C CNN "Available at"
 	1    5500 4650
 	0    1    1    0
@@
 F 3 "" V 8030 4750 50  0000 C CNN
 F 4 "1/10W" V 7870 4750 50  0000 C CNN "Power"
+F 5 "Panasonic ERJPA3F3002V (30KΩ)" V 7950 4750 60  0001 C CNN "Model"
+F 6 "http://jp.rs-online.com/web/p/products/8626896/" V 7950 4750 60  0001 C CNN "Available at"
 	1    7950 4750
 	-1   0    0    1
@@
 F 3 "" H 7600 5600 50  0000 C CNN
 F 4 "10V" H 7580 5520 50  0000 R CNN "Voltage"
+F 5 "GRM188F11H224ZA01" H 7600 5600 60  0001 C CNN "Model"
+F 6 "http://akizukidenshi.com/catalog/g/gP-05624/" H 7600 5600 60  0001 C CNN "Available at"
 	1    7600 5600
 	0    1    1    0
@@
 F 3 "" H 7600 5300 50  0000 C CNN
 F 4 "10V" H 7590 5220 50  0000 R CNN "Voltage"
+F 5 "GRM188R61E106MA" H 7600 5300 60  0001 C CNN "Model"
+F 6 "http://akizukidenshi.com/catalog/g/gP-07768/" H 7600 5300 60  0001 C CNN "Available at"
 	1    7600 5300
 	0    -1   -1   0
@@
 F 3 "" H 4800 4700 50  0000 C CNN
 F 4 "50V" H 4780 4620 50  0000 R CNN "Voltage"
+F 5 "GRM188F11H104ZA01" H 4800 4700 60  0001 C CNN "Model"
+F 6 "http://akizukidenshi.com/catalog/g/gP-04940/" H 4800 4700 60  0001 C CNN "Available at"
 	1    4800 4700
 	-1   0    0    1
@@
 F 4 "50V" H 6890 3020 50  0000 R CNN "Voltage"
 F 5 "Nichicon UCB1H101MNL1GS" H 6900 3100 60  0001 C CNN "Model"
-F 6 "RS 280yen for 10." H 6900 3100 60  0001 C CNN "Available at"
+F 6 "http://jp.rs-online.com/web/p/products/0269329/" H 6900 3100 60  0001 C CNN "Available at"
 	1    6900 3100
 	0    -1   -1   0
@@
 F 3 "" H 6900 3350 50  0000 C CNN
 F 4 "50V" H 6880 3270 50  0000 R CNN "Voltage"
+F 5 "GRM188F11H224ZA01" H 6900 3350 60  0001 C CNN "Model"
+F 6 "http://akizukidenshi.com/catalog/g/gP-05624/" H 6900 3350 60  0001 C CNN "Available at"
 	1    6900 3350
 	0    1    1    0
@@
 F 3 "" H 5100 4950 50  0000 C CNN
 F 4 "25V" H 5080 4870 50  0000 R CNN "Voltage"
+F 5 "GRM188F11H224ZA01" H 5100 4950 60  0001 C CNN "Model"
+F 6 "http://akizukidenshi.com/catalog/g/gP-05624/" H 5100 4950 60  0001 C CNN "Available at"
 	1    5100 4950
 	0    1    1    0
@@
 F 2 "Housings_SOIC:SOIC-24W_7.5x15.4mm_Pitch1.27mm" H 6500 4550 60  0001 C CNN
 F 3 "" H 6500 4550 60  0001 C CNN
+F 4 "A3982SLBTR-T" H 6400 4500 60  0001 C CNN "Model"
+F 5 "http://akizukidenshi.com/catalog/g/gI-06739/" H 6400 4500 60  0001 C CNN "Available at"
 	1    6400 4500
 	1    0    0    -1
